File: RIAA_PHONO.kicad_sch (KiCad schematic)
At the start: 21 parts, among them U1 OPA1644AxD, U2 OPA1612AxD

Commit message: CHANGE POWER SUPPLY
Parts:
- R4: renamed from R16; value 10k -> 16k
- R8: renamed from R20; value 100R -> 300R
- renumbered C7 to C1, C8 to C2, C9 to C3, C10 to C4, C11 to C5, C12 to C6, R13 to R1, R22 to R10, R23 to R11, R24 to R12, R14 to R2, R15 to R3, R17 to R5, R18 to R6, R19 to R7, R21 to R9
Connections:
- net IN2 renamed RIAA
- net IN2_R renamed RIAA_R
- net IN2_RC renamed RIAA_RC
Other:
- note added: "5mV typical"
- note added: "Gain = 22dB"
- note added: "Gain = 30dB"
- note added: "RIAA ±0.2dB - 0.6 dB @ 20 Hz -20.0 dB @ 1k Hz -40.0 dB @ 20k Hz"
- note added: "Total Gain 32dB@1kHz"
- moved on the sheet: C1, C2, C3, C4, C5, C6, R1, R10, R11, R12, R2, R3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

Commit message: update layout
Connections:
- net FB3 renamed FBTRIM
- net OUT3 renamed TRIM
Changed lines of the file:
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@@
     (effects (font (size 1.27 1.27)) (justify left bottom))
   )
-  (label "FB3" (at 229.87 106.68 0)
+  (label "FBTRIM" (at 229.87 106.68 0)
     (effects (font (size 1.27 1.27)) (justify left bottom))
   )
@@
     (effects (font (size 1.27 1.27)) (justify left bottom))
   )
-  (label "OUT3" (at 209.55 104.14 0)
+  (label "TRIM" (at 207.01 104.14 0)
     (effects (font (size 1.27 1.27)) (justify left bottom))
   )

Commit message: add usb c connector
Parts:
- renumbered C4 to C10, C5 to C11, C6 to C12, C1 to C7, C2 to C8, C3 to C9, R1 to R13, R2 to R14, R3 to R15, R4 to R16, R5 to R17, R6 to R18, R7 to R19, R8 to R20, R9 to R21, R10 to R22, R11 to R23, R12 to R24
Changed lines of the file:
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@@
       (effects (font (size 1.27 1.27)) hide)
     )
-    (pin "12")
-    (pin "13")
-    (pin "14")
+    (pin "1")
+    (pin "2")
+    (pin "3")
   )
   (symbol (lib_id "power:GND") (at 240.03 125.73 0)
@@
       (effects (font (size 1.27 1.27)) hide)
     )
-    (pin "1")
-    (pin "2")
-    (pin "3")
+    (pin "5")
+    (pin "6")
+    (pin "7")
   )
   (symbol (lib_id "Device:C") (at 240.03 120.65 0)
     (in_bom yes) (on_board yes) (fields_autoplaced)
-    (property "Reference" "C6" (id 0) (at 243.84 119.3799 0)
+    (property "Reference" "C12" (id 0) (at 243.84 119.3799 0)
       (effects (font (size 1.27 1.27)) (justify left))
     )
@@
   (symbol (lib_id "Device:R_US") (at 124.46 88.9 180)
     (in_bom yes) (on_board yes) (fields_autoplaced)
-    (property "Reference" "R5" (id 0) (at 127 87.6299 0)
+    (property "Reference" "R17" (id 0) (at 127 87.6299 0)
       (effects (font (size 1.27 1.27)) (justify right))
     )
@@
   (symbol (lib_id "Device:R_US") (at 50.8 86.36 180)
     (in_bom yes) (on_board yes) (fields_autoplaced)
-    (property "Reference" "R1" (id 0) (at 53.34 85.0899 0)
+    (property "Reference" "R13" (id 0) (at 53.34 85.0899 0)
       (effects (font (size 1.27 1.27)) (justify right))
     )
@@
   (symbol (lib_id "Device:R_US") (at 83.82 105.41 180)
     (in_bom yes) (on_board yes) (fields_autoplaced)
-    (property "Reference" "R3" (id 0) (at 86.36 104.1399 0)
+    (property "Reference" "R15" (id 0) (at 86.36 104.1399 0)
       (effects (font (size 1.27 1.27)) (justify right))
     )
@@
   (symbol (lib_id "Device:C") (at 124.46 106.68 0)
     (in_bom yes) (on_board yes) (fields_autoplaced)
-    (property "Reference" "C2" (id 0) (at 128.27 105.4099 0)
+    (property "Reference" "C8" (id 0) (at 128.27 105.4099 0)
       (effects (font (size 1.27 1.27)) (justify left))
     )
@@
   (symbol (lib_id "Device:C") (at 114.3 106.68 0)
     (in_bom yes) (on_board yes) (fields_autoplaced)
-    (property "Reference" "C4" (id 0) (at 117.475 105.4099 0)
+    (property "Reference" "C10" (id 0) (at 117.475 105.4099 0)
       (effects (font (size 1.27 1.27)) (justify left))
     )
@@
   (symbol (lib_id "Device:R_US") (at 194.31 91.44 0)
     (in_bom yes) (on_board yes) (fields_autoplaced)
-    (property "Reference" "R7" (id 0) (at 196.85 90.1699 0)
+    (property "Reference" "R19" (id 0) (at 196.85 90.1699 0)
       (effects (font (size 1.27 1.27)) (justify left))
     )
@@
   (symbol (lib_id "Device:R_US") (at 203.2 104.14 270)
     (in_bom yes) (on_board yes) (fields_autoplaced)
-    (property "Reference" "R9" (id 0) (at 203.2 97.79 90))
+    (property "Reference" "R21" (id 0) (at 203.2 97.79 90))
     (property "Value" "27.4k" (id 1) (at 203.2 100.33 90))
     (property "Footprint" "Resistor_SMD:R_0402_1005Metric" (id 2) (at 202.946 105.156 90)
@@
   (symbol (lib_id "Device:C") (at 41.91 86.36 0)
     (in_bom yes) (on_board yes) (fields_autoplaced)
-    (property "Reference" "C1" (id 0) (at 45.72 85.0899 0)
+    (property "Reference" "C7" (id 0) (at 45.72 85.0899 0)
       (effects (font (size 1.27 1.27)) (justify left))
     )
@@
   (symbol (lib_id "Device:R_US") (at 124.46 97.79 0)
     (in_bom yes) (on_board yes) (fields_autoplaced)
-    (property "Reference" "R6" (id 0) (at 127 96.5199 0)
+    (property "Reference" "R18" (id 0) (at 127 96.5199 0)
       (effects (font (size 1.27 1.27)) (justify left))
     )
@@
   (symbol (lib_id "Device:C") (at 217.17 115.57 90)
     (in_bom yes) (on_board yes) (fields_autoplaced)
-    (property "Reference" "C5" (id 0) (at 217.17 107.95 90))
+    (property "Reference" "C11" (id 0) (at 217.17 107.95 90))
     (property "Value" "470n" (id 1) (at 217.17 110.49 90))
     (property "Footprint" "Capacitor_SMD:C_0402_1005Metric" (id 2) (at 220.98 114.6048 0)
@@
       (effects (font (size 1.27 1.27)) hide)
     )
-    (pin "10")
-    (pin "8")
-    (pin "9")
+    (pin "5")
+    (pin "6")
+    (pin "7")
   )
   (symbol (lib_id "Device:R_US") (at 229.87 120.65 180)
     (in_bom yes) (on_board yes)
-    (property "Reference" "R10" (id 0) (at 232.41 119.3799 0)
+    (property "Reference" "R22" (id 0) (at 232.41 119.3799 0)
       (effects (font (size 1.27 1.27)) (justify right))
     )
@@
   (symbol (lib_id "Device:R_US") (at 194.31 110.49 180)
     (in_bom yes) (on_board yes) (fields_autoplaced)
-    (property "Reference" "R8" (id 0) (at 196.85 109.2199 0)
+    (property "Reference" "R20" (id 0) (at 196.85 109.2199 0)
       (effects (font (size 1.27 1.27)) (justify right))
     )
@@
   (symbol (lib_id "Device:R_US") (at 240.03 93.98 0)
     (in_bom yes) (on_board yes) (fields_autoplaced)
-    (property "Reference" "R11" (id 0) (at 242.57 92.7099 0)
+    (property "Reference" "R23" (id 0) (at 242.57 92.7099 0)
       (effects (font (size 1.27 1.27)) (justify left))
     )
@@
   (symbol (lib_id "Device:R_US") (at 83.82 91.44 0)
     (in_bom yes) (on_board yes) (fields_autoplaced)
-    (property "Reference" "R2" (id 0) (at 86.36 90.1699 0)
+    (property "Reference" "R14" (id 0) (at 86.36 90.1699 0)
       (effects (font (size 1.27 1.27)) (justify left))
     )
@@
   (symbol (lib_id "Device:R_US") (at 109.22 83.82 270)
     (in_bom yes) (on_board yes) (fields_autoplaced)
-    (property "Reference" "R4" (id 0) (at 109.22 77.47 90))
+    (property "Reference" "R16" (id 0) (at 109.22 77.47 90))
     (property "Value" "16k" (id 1) (at 109.22 80.01 90))
     (property "Footprint" "Resistor_SMD:R_0402_1005Metric" (id 2) (at 108.966 84.836 90)
@@
   (symbol (lib_id "Device:C") (at 137.16 106.68 0)
     (in_bom yes) (on_board yes)
-    (property "Reference" "C3" (id 0) (at 140.97 105.4099 0)
+    (property "Reference" "C9" (id 0) (at 140.97 105.4099 0)
       (effects (font (size 1.27 1.27)) (justify left))
     )
@@
   (symbol (lib_id "Device:R_US") (at 250.19 86.36 90)
     (in_bom yes) (on_board yes) (fields_autoplaced)
-    (property "Reference" "R12" (id 0) (at 250.19 80.01 90))
+    (property "Reference" "R24" (id 0) (at 250.19 80.01 90))
     (property "Value" "100R" (id 1) (at 250.19 82.55 90))
     (property "Footprint" "Resistor_SMD:R_0402_1005Metric" (id 2) (at 250.444 85.344 90)

Commit message: Update component fields
Parts:
- C2: renamed from C8; footprint Capacitor_SMD:C_1206_3216Metric -> Capacitor_SMD:C_1210_3225Metric; MPN (none) -> ECH-U1C683GX5; Manufacturer (none) -> Panasonic Electronic Components
- C3: renamed from C9; footprint Capacitor_SMD:C_1206_3216Metric -> Capacitor_SMD:C_1210_3225Metric; MPN (none) -> ECH-U1C683GX5; Manufacturer (none) -> Panasonic Electronic Components
- C4: renamed from C10; MPN (none) -> ECH-U1C473GX5; Manufacturer (none) -> Panasonic Electronic Components
- R1: renamed from R13; value R_US -> 47k; MPN (none) -> RT0402DRE0747KL; Manufacturer (none) -> YAGEO
- R10: renamed from R22; MPN (none) -> RC0402FR-07470KL; Manufacturer (none) -> YAGEO
- R11: renamed from R23; MPN (none) -> RC0402FR-07470KL; Manufacturer (none) -> YAGEO
- R12: renamed from R24; MPN (none) -> RT0402DRE07100RL; Manufacturer (none) -> YAGEO
- R2: renamed from R14; MPN (none) -> RT0402FRE073K3L; Manufacturer (none) -> YAGEO
- R3: renamed from R15; MPN (none) -> RT0402DRE07100RL; Manufacturer (none) -> YAGEO
- R4: renamed from R16; MPN (none) -> RT0402FRE0716KL; Manufacturer (none) -> YAGEO
- R5: renamed from R17; MPN (none) -> MCS04020C2201FE000; Manufacturer (none) -> VISHAY
- R6: renamed from R18; MPN (none) -> RT0402BRD07127RL; Manufacturer (none) -> YAGEO
- R7: renamed from R19; MPN (none) -> RT0402FRE073K3L; Manufacturer (none) -> YAGEO
- R8: renamed from R20; MPN (none) -> RT0402FRE07300RL; Manufacturer (none) -> YAGEO
- R9: renamed from R21; MPN (none) -> RT0402FRE0727K4L; Manufacturer (none) -> YAGEO
- U1: MPN (none) -> OPA1644AID; Manufacturer (none) -> Texas Instruments
- U2: MPN (none) -> OPA1612AID; Manufacturer (none) -> Texas Instruments
- renumbered C7 to C1, C11 to C5, C12 to C6

Commit message: routed all nets
Parts:
- C11: renamed from C5; value 470n -> 1u; MPN (none) -> GRM155R61E105KA12D; Manufacturer (none) -> Murata Electronics
- C12: renamed from C6; value 470n -> 1u; MPN (none) -> GRM155R61E105KA12D; Manufacturer (none) -> Murata Electronics
- C7: renamed from C1; value C -> NP; now left out of the parts list
- renumbered C4 to C10, C2 to C8, C3 to C9, R1 to R13, R2 to R14, R3 to R15, R4 to R16, R5 to R17, R6 to R18, R7 to R19, R8 to R20, R9 to R21, R10 to R22, R11 to R23, R12 to R24
Other:
- note added: "C1/C7 Select per cartridge loading"

Commit message: Clean DRC
Parts:
- renumbered C7 to C1, C8 to C2, C9 to C3, C10 to C4, C11 to C5, C12 to C6, R13 to R1, R22 to R10, R23 to R11, R24 to R12, R14 to R2, R15 to R3, R16 to R4, R17 to R5, R18 to R6, R19 to R7, R20 to R8, R21 to R9
Changed lines of the file:
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@@
       (effects (font (size 1.27 1.27)) hide)
     )
-    (pin "5")
-    (pin "6")
-    (pin "7")
+    (pin "1")
+    (pin "2")
+    (pin "3")
   )
   (symbol (lib_id "Device:C") (at 240.03 120.65 0)
     (in_bom yes) (on_board yes) (fields_autoplaced)
-    (property "Reference" "C12" (id 0) (at 243.84 119.3799 0)
+    (property "Reference" "C6" (id 0) (at 243.84 119.3799 0)
       (effects (font (size 1.27 1.27)) (justify left))
     )
@@
   (symbol (lib_id "Device:R_US") (at 124.46 88.9 180)
     (in_bom yes) (on_board yes) (fields_autoplaced)
-    (property "Reference" "R17" (id 0) (at 127 87.6299 0)
+    (property "Reference" "R5" (id 0) (at 127 87.6299 0)
       (effects (font (size 1.27 1.27)) (justify right))
     )
@@
   (symbol (lib_id "Device:R_US") (at 50.8 86.36 180)
     (in_bom yes) (on_board yes) (fields_autoplaced)
-    (property "Reference" "R13" (id 0) (at 53.34 85.0899 0)
+    (property "Reference" "R1" (id 0) (at 53.34 85.0899 0)
       (effects (font (size 1.27 1.27)) (justify right))
     )
@@
   (symbol (lib_id "Device:R_US") (at 83.82 105.41 180)
     (in_bom yes) (on_board yes) (fields_autoplaced)
-    (property "Reference" "R15" (id 0) (at 86.36 104.1399 0)
+    (property "Reference" "R3" (id 0) (at 86.36 104.1399 0)
       (effects (font (size 1.27 1.27)) (justify right))
     )
@@
   (symbol (lib_id "Device:C") (at 124.46 106.68 0)
     (in_bom yes) (on_board yes) (fields_autoplaced)
-    (property "Reference" "C8" (id 0) (at 128.27 105.4099 0)
+    (property "Reference" "C2" (id 0) (at 128.27 105.4099 0)
       (effects (font (size 1.27 1.27)) (justify left))
     )
@@
   (symbol (lib_id "Device:C") (at 114.3 106.68 0)
     (in_bom yes) (on_board yes) (fields_autoplaced)
-    (property "Reference" "C10" (id 0) (at 117.475 105.4099 0)
+    (property "Reference" "C4" (id 0) (at 117.475 105.4099 0)
       (effects (font (size 1.27 1.27)) (justify left))
     )
@@
   (symbol (lib_id "Device:R_US") (at 194.31 91.44 0)
     (in_bom yes) (on_board yes) (fields_autoplaced)
-    (property "Reference" "R19" (id 0) (at 196.85 90.1699 0)
+    (property "Reference" "R7" (id 0) (at 196.85 90.1699 0)
       (effects (font (size 1.27 1.27)) (justify left))
     )
@@
   (symbol (lib_id "Device:R_US") (at 203.2 104.14 270)
     (in_bom yes) (on_board yes) (fields_autoplaced)
-    (property "Reference" "R21" (id 0) (at 203.2 97.79 90))
+    (property "Reference" "R9" (id 0) (at 203.2 97.79 90))
     (property "Value" "27.4k" (id 1) (at 203.2 100.33 90))
     (property "Footprint" "Resistor_SMD:R_0402_1005Metric" (id 2) (at 202.946 105.156 90)
@@
   (symbol (lib_id "Device:C") (at 41.91 86.36 0)
     (in_bom no) (on_board yes) (fields_autoplaced)
-    (property "Reference" "C7" (id 0) (at 45.72 85.0899 0)
+    (property "Reference" "C1" (id 0) (at 45.72 85.0899 0)
       (effects (font (size 1.27 1.27)) (justify left))
     )
@@
   (symbol (lib_id "Device:R_US") (at 124.46 97.79 0)
     (in_bom yes) (on_board yes) (fields_autoplaced)
-    (property "Reference" "R18" (id 0) (at 127 96.5199 0)
+    (property "Reference" "R6" (id 0) (at 127 96.5199 0)
       (effects (font (size 1.27 1.27)) (justify left))
     )
@@
   (symbol (lib_id "Device:C") (at 217.17 115.57 90)
     (in_bom yes) (on_board yes) (fields_autoplaced)
-    (property "Reference" "C11" (id 0) (at 217.17 107.95 90))
+    (property "Reference" "C5" (id 0) (at 217.17 107.95 90))
     (property "Value" "1u" (id 1) (at 217.17 110.49 90))
     (property "Footprint" "Capacitor_SMD:C_0402_1005Metric" (id 2) (at 220.98 114.6048 0)
@@
       (effects (font (size 1.27 1.27)) hide)
     )
-    (pin "5")
-    (pin "6")
-    (pin "7")
+    (pin "1")
+    (pin "2")
+    (pin "3")
   )
   (symbol (lib_id "Device:R_US") (at 229.87 120.65 180)
     (in_bom yes) (on_board yes)
-    (property "Reference" "R22" (id 0) (at 232.41 119.3799 0)
+    (property "Reference" "R10" (id 0) (at 232.41 119.3799 0)
       (effects (font (size 1.27 1.27)) (justify right))
     )
@@
   (symbol (lib_id "Device:R_US") (at 194.31 110.49 180)
     (in_bom yes) (on_board yes) (fields_autoplaced)
-    (property "Reference" "R20" (id 0) (at 196.85 109.2199 0)
+    (property "Reference" "R8" (id 0) (at 196.85 109.2199 0)
       (effects (font (size 1.27 1.27)) (justify right))
     )
@@
   (symbol (lib_id "Device:R_US") (at 240.03 93.98 0)
     (in_bom yes) (on_board yes) (fields_autoplaced)
-    (property "Reference" "R23" (id 0) (at 242.57 92.7099 0)
+    (property "Reference" "R11" (id 0) (at 242.57 92.7099 0)
       (effects (font (size 1.27 1.27)) (justify left))
     )
@@
   (symbol (lib_id "Device:R_US") (at 83.82 91.44 0)
     (in_bom yes) (on_board yes) (fields_autoplaced)
-    (property "Reference" "R14" (id 0) (at 86.36 90.1699 0)
+    (property "Reference" "R2" (id 0) (at 86.36 90.1699 0)
       (effects (font (size 1.27 1.27)) (justify left))
     )
@@
   (symbol (lib_id "Device:R_US") (at 109.22 83.82 270)
     (in_bom yes) (on_board yes) (fields_autoplaced)
-    (property "Reference" "R16" (id 0) (at 109.22 77.47 90))
+    (property "Reference" "R4" (id 0) (at 109.22 77.47 90))
     (property "Value" "16k" (id 1) (at 109.22 80.01 90))
     (property "Footprint" "Resistor_SMD:R_0402_1005Metric" (id 2) (at 108.966 84.836 90)
@@
   (symbol (lib_id "Device:C") (at 137.16 106.68 0)
     (in_bom yes) (on_board yes)
-    (property "Reference" "C9" (id 0) (at 140.97 105.4099 0)
+    (property "Reference" "C3" (id 0) (at 140.97 105.4099 0)
       (effects (font (size 1.27 1.27)) (justify left))
     )
@@
   (symbol (lib_id "Device:R_US") (at 250.19 86.36 90)
     (in_bom yes) (on_board yes) (fields_autoplaced)
-    (property "Reference" "R24" (id 0) (at 250.19 80.01 90))
+    (property "Reference" "R12" (id 0) (at 250.19 80.01 90))
     (property "Value" "100R" (id 1) (at 250.19 82.55 90))
     (property "Footprint" "Resistor_SMD:R_0402_1005Metric" (id 2) (at 250.444 85.344 90)

Commit message: simplify BOM
Parts:
- removed R6: 127R, Resistor_SMD:R_0402_1005Metric, symbol Device:R_US
- C1: Size (none) -> 0402
- C2, C3: Rating (none) -> 16V; Size (none) -> 1210; Tolerance (none) -> 2%
- C4: Rating (none) -> 16V; Size (none) -> 1206; Tolerance (none) -> 2%
- C5, C6: Rating (none) -> 25V; Size (none) -> 0402; Tolerance (none) -> X5R
- R1, R12, R3: Size (none) -> 0402; Tolerance (none) -> 0.5%
- R10, R11: value 470k -> 47k; MPN RC0402FR-07470KL -> RT0402DRE0747KL; Size (none) -> 0402; Tolerance (none) -> 0.5%
- R2, R4, R7: Size (none) -> 0402; Tolerance (none) -> 1%
- R5: value 2.2k -> 2.32k; MPN MCS04020C2201FE000 -> RT0402BRD072K32L; Manufacturer VISHAY -> YAGEO; Size (none) -> 0402; Tolerance (none) -> 1%
- R8: value 300R -> 100R; MPN RT0402FRE07300RL -> RT0402DRE07100RL; Size (none) -> 0402; Tolerance (none) -> 0.5%
- R9: value 27.4k -> 47k; MPN RT0402FRE0727K4L -> RT0402DRE0747KL; Size (none) -> 0402; Tolerance (none) -> 0.5%
Connections:
- net RIAA_R is gone; now on net RIAA_RC: R5.1
Other:
- note added: "Total Gain 40dB@1kHz"
- note removed: "Gain = 22dB"
- note removed: "Total Gain 32dB@1kHz"

Commit message: Add graphics, simplify output resistor
Parts:
- R13: renamed from R1; MPN RT0402DRE0747KL -> RT0402FRE0747KL; Tolerance 0.5% -> 1%
- R14: renamed from R2; value 3.3k -> 2.32k; MPN RT0402FRE073K3L -> RT0402FRE072K32L
- R15: renamed from R3; value 100R -> 68R; MPN RT0402DRE07100RL -> RT0402FRE0768RL; Tolerance 0.5% -> 1%
- R17: renamed from R5; MPN RT0402BRD072K32L -> RT0402FRE072K32L
- R19: renamed from R7; value 3.3k -> 2.32k; MPN RT0402FRE073K3L -> RT0402FRE072K32L
- R21: renamed from R9; MPN RT0402DRE0747KL -> RT0402FRE0747KL; Tolerance 0.5% -> 1%
- R22: renamed from R10; MPN RT0402DRE0747KL -> RT0402FRE0747KL; Tolerance 0.5% -> 1%
- R23: renamed from R11; MPN RT0402DRE0747KL -> RT0402FRE0747KL; Tolerance 0.5% -> 1%
- R24: renamed from R12; value 100R -> 68R; MPN RT0402DRE07100RL -> RT0402FRE0768RL; Tolerance 0.5% -> 1%
- R6: renamed from R8; value 100R -> 68R; MPN RT0402DRE07100RL -> RT0402FRE0768RL; Tolerance 0.5% -> 1%
- renumbered C4 to C10, C5 to C11, C6 to C12, C1 to C7, C2 to C8, C3 to C9, R4 to R16
Other:
- note added: "Gain = 31dB"
- note added: "Total Gain 42dB@1kHz"
- note removed: "Gain = 30dB"
- note removed: "Total Gain 40dB@1kHz"
