File: RIAA_PHONO.kicad_sch (KiCad schematic)
At the start: 20 parts, among them U1 OPA1644AxD, U2 OPA1612AxD

Commit message: change output resistor to 499R
Parts:
- R14, R19: value 2.32k -> 16k; MPN RT0402FRE072K32L -> RT0402FRE0716KL
- R15, R24, R6: value 68R -> 499R; MPN RT0402FRE0768RL -> RT0402FRE07499RL
Other:
- note added: "Gain = 30dB"
- note added: "Total Gain 40dB@1kHz"
- note removed: "Gain = 31dB"
- note removed: "Total Gain 42dB@1kHz"
Changed lines of the file:
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@@
     (effects (font (size 1.27 1.27)) (justify left bottom))
   )
-  (text "Total Gain 42dB@1kHz" (at 250.19 91.44 0)
+  (text "Total Gain 40dB@1kHz" (at 250.19 91.44 0)
     (effects (font (size 1.27 1.27)) (justify left bottom))
   )
@@
     (effects (font (size 1.27 1.27)) (justify left bottom))
   )
-  (text "Gain = 31dB" (at 64.77 97.79 0)
-    (effects (font (size 1.27 1.27)) (justify left bottom))
-  )
-  (text "Gain = 31dB" (at 175.26 97.79 0)
+  (text "Gain = 30dB" (at 64.77 97.79 0)
+    (effects (font (size 1.27 1.27)) (justify left bottom))
+  )
+  (text "Gain = 30dB" (at 175.26 97.79 0)
     (effects (font (size 1.27 1.27)) (justify left bottom))
   )
@@
       (effects (font (size 1.27 1.27)) (justify right))
     )
-    (property "Value" "68R" (id 1) (at 86.36 106.6799 0)
+    (property "Value" "499R" (id 1) (at 86.36 106.6799 0)
       (effects (font (size 1.27 1.27)) (justify right))
     )
@@
       (effects (font (size 1.27 1.27)) hide)
     )
-    (property "Description" "RES SMD 68 OHM 1% 1/16W 0402" (id 4) (at 83.82 105.41 0)
-      (effects (font (size 1.27 1.27)) hide)
-    )
-    (property "MPN" "RT0402FRE0768RL" (id 5) (at 83.82 105.41 0)
+    (property "Description" "RES SMD 499R OHM 1% 1/16W 0402" (id 4) (at 83.82 105.41 0)
+      (effects (font (size 1.27 1.27)) hide)
+    )
+    (property "MPN" "RT0402FRE07499RL" (id 5) (at 83.82 105.41 0)
       (effects (font (size 1.27 1.27)) hide)
     )
@@
       (effects (font (size 1.27 1.27)) (justify left))
     )
-    (property "Value" "2.32k" (id 1) (at 196.85 92.7099 0)
+    (property "Value" "16k" (id 1) (at 196.85 92.7099 0)
       (effects (font (size 1.27 1.27)) (justify left))
     )
@@
       (effects (font (size 1.27 1.27)) hide)
     )
-    (property "Description" "RES SMD 2.32K OHM 1% 1/16W 0402" (id 4) (at 194.31 91.44 0)
-      (effects (font (size 1.27 1.27)) hide)
-    )
-    (property "MPN" "RT0402FRE072K32L" (id 5) (at 194.31 91.44 0)
+    (property "Description" "RES SMD 16K OHM 1% 1/16W 0402" (id 4) (at 194.31 91.44 0)
+      (effects (font (size 1.27 1.27)) hide)
+    )
+    (property "MPN" "RT0402FRE0716KL" (id 5) (at 194.31 91.44 0)
       (effects (font (size 1.27 1.27)) hide)
     )
@@
       (effects (font (size 1.27 1.27)) (justify left))
     )
-    (property "Value" "2.32k" (id 1) (at 86.36 92.7099 0)
+    (property "Value" "16k" (id 1) (at 86.36 92.7099 0)
       (effects (font (size 1.27 1.27)) (justify left))
     )
@@
       (effects (font (size 1.27 1.27)) hide)
     )
-    (property "Description" "RES SMD 2.32K OHM 1% 1/16W 0402" (id 4) (at 83.82 91.44 0)
-      (effects (font (size 1.27 1.27)) hide)
-    )
-    (property "MPN" "RT0402FRE072K32L" (id 5) (at 83.82 91.44 0)
+    (property "Description" "RES SMD 16K OHM 1% 1/16W 0402" (id 4) (at 83.82 91.44 0)
+      (effects (font (size 1.27 1.27)) hide)
+    )
+    (property "MPN" "RT0402FRE0716KL" (id 5) (at 83.82 91.44 0)
       (effects (font (size 1.27 1.27)) hide)
     )
@@
       (effects (font (size 1.27 1.27)) (justify right))
     )
-    (property "Value" "68R" (id 1) (at 196.85 111.7599 0)
+    (property "Value" "499R" (id 1) (at 196.85 111.7599 0)
       (effects (font (size 1.27 1.27)) (justify right))
     )
@@
       (effects (font (size 1.27 1.27)) hide)
     )
-    (property "Description" "RES SMD 68 OHM 1% 1/16W 0402" (id 4) (at 194.31 110.49 0)
-      (effects (font (size 1.27 1.27)) hide)
-    )
-    (property "MPN" "RT0402FRE0768RL" (id 5) (at 194.31 110.49 0)
+    (property "Description" "RES SMD 499R OHM 1% 1/16W 0402" (id 4) (at 194.31 110.49 0)
+      (effects (font (size 1.27 1.27)) hide)
+    )
+    (property "MPN" "RT0402FRE07499RL" (id 5) (at 194.31 110.49 0)
       (effects (font (size 1.27 1.27)) hide)
     )
@@
     (in_bom yes) (on_board yes) (fields_autoplaced)
     (property "Reference" "R24" (id 0) (at 250.19 80.01 90))
-    (property "Value" "68R" (id 1) (at 250.19 82.55 90))
+    (property "Value" "499R" (id 1) (at 250.19 82.55 90))
     (property "Footprint" "Resistor_SMD:R_0402_1005Metric" (id 2) (at 250.444 85.344 90)
       (effects (font (size 1.27 1.27)) hide)
@@
       (effects (font (size 1.27 1.27)) hide)
     )
-    (property "Description" "RES SMD 68 OHM 1% 1/16W 0402" (id 4) (at 250.19 86.36 0)
-      (effects (font (size 1.27 1.27)) hide)
-    )
-    (property "MPN" "RT0402FRE0768RL" (id 5) (at 250.19 86.36 0)
-      (effects (font (size 1.27 1.27)) hide)
-    )
+    (property "Description" "RES SMD 499R OHM 1% 1/16W 0402" (id 4) (at 250.19 86.36 0)
+      (effects (font (size 1.27 1.27)) hide)
+    )
+    (property "MPN" "RT0402FRE07499RL" (id 5) (at 250.19 86.36 0)
+      (effects (font (size 1.27 1.27)) hide)
+    )

Commit message: Generate Gerbers
Parts:
- renumbered C7 to C1, C8 to C2, C9 to C3, C10 to C4, C11 to C5, C12 to C6, R13 to R1, R22 to R10, R23 to R11, R24 to R12, R14 to R2, R15 to R3, R16 to R4, R17 to R5, R19 to R7, R6 to R8, R21 to R9
Changed lines of the file:
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@@
       (effects (font (size 1.27 1.27)) hide)
     )
-    (pin "1")
-    (pin "2")
-    (pin "3")
+    (pin "12")
+    (pin "13")
+    (pin "14")
   )
   (symbol (lib_id "power:GND") (at 240.03 125.73 0)
     (in_bom yes) (on_board yes) (fields_autoplaced)
-    (property "Reference" "#PWR020" (id 0) (at 240.03 132.08 0)
+    (property "Reference" "#PWR012" (id 0) (at 240.03 132.08 0)
       (effects (font (size 1.27 1.27)) hide)
     )
@@
   (symbol (lib_id "power:GND") (at 194.31 115.57 0)
     (in_bom yes) (on_board yes) (fields_autoplaced)
-    (property "Reference" "#PWR018" (id 0) (at 194.31 121.92 0)
+    (property "Reference" "#PWR010" (id 0) (at 194.31 121.92 0)
       (effects (font (size 1.27 1.27)) hide)
     )
@@
       (effects (font (size 1.27 1.27)) hide)
     )
-    (pin "5")
-    (pin "6")
-    (pin "7")
+    (pin "1")
+    (pin "2")
+    (pin "3")
   )
   (symbol (lib_id "Device:C") (at 240.03 120.65 0)
     (in_bom yes) (on_board yes) (fields_autoplaced)
-    (property "Reference" "C12" (id 0) (at 243.84 119.3799 0)
+    (property "Reference" "C6" (id 0) (at 243.84 119.3799 0)
       (effects (font (size 1.27 1.27)) (justify left))
     )
@@
   (symbol (lib_id "Device:R_US") (at 124.46 88.9 180)
     (in_bom yes) (on_board yes) (fields_autoplaced)
-    (property "Reference" "R17" (id 0) (at 127 87.6299 0)
+    (property "Reference" "R5" (id 0) (at 127 87.6299 0)
       (effects (font (size 1.27 1.27)) (justify right))
     )
@@
   (symbol (lib_id "Device:R_US") (at 50.8 86.36 180)
     (in_bom yes) (on_board yes) (fields_autoplaced)
-    (property "Reference" "R13" (id 0) (at 53.34 85.0899 0)
+    (property "Reference" "R1" (id 0) (at 53.34 85.0899 0)
       (effects (font (size 1.27 1.27)) (justify right))
     )
@@
   (symbol (lib_id "Device:R_US") (at 83.82 105.41 180)
     (in_bom yes) (on_board yes) (fields_autoplaced)
-    (property "Reference" "R15" (id 0) (at 86.36 104.1399 0)
+    (property "Reference" "R3" (id 0) (at 86.36 104.1399 0)
       (effects (font (size 1.27 1.27)) (justify right))
     )
@@
   (symbol (lib_id "Device:C") (at 124.46 106.68 0)
     (in_bom yes) (on_board yes) (fields_autoplaced)
-    (property "Reference" "C8" (id 0) (at 128.27 105.4099 0)
+    (property "Reference" "C2" (id 0) (at 128.27 105.4099 0)
       (effects (font (size 1.27 1.27)) (justify left))
     )
@@
   (symbol (lib_id "power:GND") (at 229.87 125.73 0)
     (in_bom yes) (on_board yes) (fields_autoplaced)
-    (property "Reference" "#PWR019" (id 0) (at 229.87 132.08 0)
+    (property "Reference" "#PWR011" (id 0) (at 229.87 132.08 0)
       (effects (font (size 1.27 1.27)) hide)
     )
@@
   (symbol (lib_id "Device:C") (at 114.3 106.68 0)
     (in_bom yes) (on_board yes) (fields_autoplaced)
-    (property "Reference" "C10" (id 0) (at 117.475 105.4099 0)
+    (property "Reference" "C4" (id 0) (at 117.475 105.4099 0)
       (effects (font (size 1.27 1.27)) (justify left))
     )
@@
   (symbol (lib_id "Device:R_US") (at 194.31 91.44 0)
     (in_bom yes) (on_board yes) (fields_autoplaced)
-    (property "Reference" "R19" (id 0) (at 196.85 90.1699 0)
+    (property "Reference" "R7" (id 0) (at 196.85 90.1699 0)
       (effects (font (size 1.27 1.27)) (justify left))
     )
@@
   (symbol (lib_id "power:GND") (at 83.82 111.76 0)
     (in_bom yes) (on_board yes) (fields_autoplaced)
-    (property "Reference" "#PWR014" (id 0) (at 83.82 118.11 0)
+    (property "Reference" "#PWR06" (id 0) (at 83.82 118.11 0)
       (effects (font (size 1.27 1.27)) hide)
     )
@@
   (symbol (lib_id "power:GND") (at 41.91 92.71 0)
     (in_bom yes) (on_board yes) (fields_autoplaced)
-    (property "Reference" "#PWR013" (id 0) (at 41.91 99.06 0)
+    (property "Reference" "#PWR05" (id 0) (at 41.91 99.06 0)
       (effects (font (size 1.27 1.27)) hide)
     )
@@
   (symbol (lib_id "Device:R_US") (at 203.2 104.14 270)
     (in_bom yes) (on_board yes) (fields_autoplaced)
-    (property "Reference" "R21" (id 0) (at 203.2 97.79 90))
+    (property "Reference" "R9" (id 0) (at 203.2 97.79 90))
     (property "Value" "47k" (id 1) (at 203.2 100.33 90))
     (property "Footprint" "Resistor_SMD:R_0402_1005Metric" (id 2) (at 202.946 105.156 90)
@@
   (symbol (lib_id "Device:C") (at 41.91 86.36 0)
     (in_bom no) (on_board yes) (fields_autoplaced)
-    (property "Reference" "C7" (id 0) (at 45.72 85.0899 0)
+    (property "Reference" "C1" (id 0) (at 45.72 85.0899 0)
       (effects (font (size 1.27 1.27)) (justify left))
     )
@@
   (symbol (lib_id "Device:C") (at 217.17 115.57 90)
     (in_bom yes) (on_board yes) (fields_autoplaced)
-    (property "Reference" "C11" (id 0) (at 217.17 107.95 90))
+    (property "Reference" "C5" (id 0) (at 217.17 107.95 90))
     (property "Value" "1u" (id 1) (at 217.17 110.49 90))
     (property "Footprint" "Capacitor_SMD:C_0402_1005Metric" (id 2) (at 220.98 114.6048 0)
@@
   (symbol (lib_id "power:GND") (at 137.16 111.76 0)
     (in_bom yes) (on_board yes) (fields_autoplaced)
-    (property "Reference" "#PWR016" (id 0) (at 137.16 118.11 0)
+    (property "Reference" "#PWR08" (id 0) (at 137.16 118.11 0)
       (effects (font (size 1.27 1.27)) hide)
     )
@@
       (effects (font (size 1.27 1.27)) hide)
     )
-    (pin "5")
-    (pin "6")
-    (pin "7")
+    (pin "10")
+    (pin "8")
+    (pin "9")
   )
   (symbol (lib_id "Device:R_US") (at 229.87 120.65 180)
     (in_bom yes) (on_board yes)
-    (property "Reference" "R22" (id 0) (at 232.41 119.3799 0)
+    (property "Reference" "R10" (id 0) (at 232.41 119.3799 0)
       (effects (font (size 1.27 1.27)) (justify right))
     )
@@
   (symbol (lib_id "Device:R_US") (at 240.03 93.98 0)
     (in_bom yes) (on_board yes) (fields_autoplaced)
-    (property "Reference" "R23" (id 0) (at 242.57 92.7099 0)
+    (property "Reference" "R11" (id 0) (at 242.57 92.7099 0)
       (effects (font (size 1.27 1.27)) (justify left))
     )
@@
   (symbol (lib_id "Device:R_US") (at 83.82 91.44 0)
     (in_bom yes) (on_board yes) (fields_autoplaced)
-    (property "Reference" "R14" (id 0) (at 86.36 90.1699 0)
+    (property "Reference" "R2" (id 0) (at 86.36 90.1699 0)
       (effects (font (size 1.27 1.27)) (justify left))
     )
@@
   (symbol (lib_id "Device:R_US") (at 194.31 110.49 180)
     (in_bom yes) (on_board yes) (fields_autoplaced)
-    (property "Reference" "R6" (id 0) (at 196.85 109.2199 0)
+    (property "Reference" "R8" (id 0) (at 196.85 109.2199 0)
       (effects (font (size 1.27 1.27)) (justify right))
     )
@@
   (symbol (lib_id "power:GND") (at 124.46 111.76 0)
     (in_bom yes) (on_board yes) (fields_autoplaced)
-    (property "Reference" "#PWR015" (id 0) (at 124.46 118.11 0)
+    (property "Reference" "#PWR07" (id 0) (at 124.46 118.11 0)
       (effects (font (size 1.27 1.27)) hide)
     )
@@
   (symbol (lib_id "Device:R_US") (at 109.22 83.82 270)
     (in_bom yes) (on_board yes) (fields_autoplaced)
-    (property "Reference" "R16" (id 0) (at 109.22 77.47 90))
+    (property "Reference" "R4" (id 0) (at 109.22 77.47 90))
     (property "Value" "16k" (id 1) (at 109.22 80.01 90))
     (property "Footprint" "Resistor_SMD:R_0402_1005Metric" (id 2) (at 108.966 84.836 90)
@@
   (symbol (lib_id "Device:C") (at 137.16 106.68 0)
     (in_bom yes) (on_board yes)
-    (property "Reference" "C9" (id 0) (at 140.97 105.4099 0)
+    (property "Reference" "C3" (id 0) (at 140.97 105.4099 0)
       (effects (font (size 1.27 1.27)) (justify left))
     )
@@
   (symbol (lib_id "power:GND") (at 114.3 111.7153 0)
     (in_bom yes) (on_board yes) (fields_autoplaced)
-    (property "Reference" "#PWR017" (id 0) (at 114.3 118.0653 0)
+    (property "Reference" "#PWR09" (id 0) (at 114.3 118.0653 0)
       (effects (font (size 1.27 1.27)) hide)
     )
@@
   (symbol (lib_id "Device:R_US") (at 250.19 86.36 90)
     (in_bom yes) (on_board yes) (fields_autoplaced)
-    (property "Reference" "R24" (id 0) (at 250.19 80.01 90))
+    (property "Reference" "R12" (id 0) (at 250.19 80.01 90))
     (property "Value" "499R" (id 1) (at 250.19 82.55 90))
     (property "Footprint" "Resistor_SMD:R_0402_1005Metric" (id 2) (at 250.444 85.344 90)
