File: OPA_PHONO.kicad_sch (KiCad schematic)
At the start: 5 parts, among them J1 PJRAS2X1S01X, J2 PJRAS2X1S01X, J3 UJC-HP-3-SMT-TR

Commit message: Generate Gerbers
Parts:
- added N1: Housing, symbol Mechanical:Housing
Changed lines of the file:
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@@
     (pin "1")
+  )
+  (symbol (lib_id "Mechanical:Housing") (at 208.28 120.65 0) (unit 1)
+    (in_bom yes) (on_board no) (fields_autoplaced)
+    (property "Reference" "N1" (id 0) (at 212.09 119.6974 0)
+      (effects (font (size 1.27 1.27)) (justify left))
+    )
+    (property "Value" "Housing" (id 1) (at 212.09 122.2374 0)
+      (effects (font (size 1.27 1.27)) (justify left))
+    )
+    (property "Footprint" "" (id 2) (at 209.55 119.38 0)
+      (effects (font (size 1.27 1.27)) hide)
+    )
+    (property "Datasheet" "https://www.hammfg.com/files/parts/pdf/1455L801.pdf" (id 3) (at 209.55 119.38 0)
+      (effects (font (size 1.27 1.27)) hide)
+    )
+    (property "Description" "BOX ALUM NATURAL 3.15\"LX4.05\"W" (id 4) (at 208.28 120.65 0)
+      (effects (font (size 1.27 1.27)) hide)
+    )
+    (property "MPN" "1455L801" (id 5) (at 208.28 120.65 0)
+      (effects (font (size 1.27 1.27)) hide)
+    )
+    (property "Manufacturer" "Hammond Manufacturing" (id 6) (at 208.28 120.65 0)
+      (effects (font (size 1.27 1.27)) hide)
+    )
   )
   (symbol (lib_id "OPA_PHONO:PJRAS2X1S01X") (at 132.08 72.39 180) (unit 1)
@@
       (reference "C14") (unit 1) (value "1u") (footprint "Capacitor_SMD:C_0402_1005Metric")
     )
+    (path "/54617677-cfc6-4c88-8682-59d8a487d34d/5f4c7c24-0d8b-4ff9-829a-ae38833fd421"
+      (reference "C15") (unit 1) (value "10u") (footprint "Capacitor_SMD:C_0805_2012Metric")
+    )
     (path "/54617677-cfc6-4c88-8682-59d8a487d34d/47a1e06a-e776-4a90-9d1f-892164164505"
       (reference "C16") (unit 1) (value "1u") (footprint "Capacitor_SMD:C_0402_1005Metric")
@@
       (reference "C24") (unit 1) (value "10u") (footprint "Capacitor_SMD:C_0805_2012Metric")
     )
+    (path "/54617677-cfc6-4c88-8682-59d8a487d34d/eb3b75c6-f775-48c1-aa10-2016bd53ab26"
+      (reference "C25") (unit 1) (value "10u") (footprint "Capacitor_SMD:C_0805_2012Metric")
+    )
     (path "/54617677-cfc6-4c88-8682-59d8a487d34d/398fdf8b-e7c5-4505-87b4-8312a52709d4"
       (reference "C26") (unit 1) (value "10u") (footprint "Capacitor_SMD:C_0805_2012Metric")
@@
       (reference "J3") (unit 1) (value "UJC-HP-3-SMT-TR") (footprint "OPA_PHONO:CUI_UJC-HP-3-SMT-TR")
     )
+    (path "/f85b707b-c164-44fe-b6f5-1f0641c164e8"
+      (reference "N1") (unit 1) (value "Housing") (footprint "")
+    )
     (path "/b71452ae-e2ec-4238-9d16-71d9677f964c/2a4ad1e3-8d24-4e7f-868b-1019aa3d2553"
