File: POWER.kicad_sch (KiCad schematic)
At the start: 23 parts, among them U1 OPA1644AxD, U2 OPA1612AxD, U3 LT3032-12

Commit message: CHANGE POWER SUPPLY
Parts:
- removed C23, C24, C25, C26: 2200uF, Capacitor_SMD:CP_Elec_18x17.5, symbol Device:C_Polarized_US
- removed C27, C28: 1u, Capacitor_SMD:C_0402_1005Metric, symbol Device:C
- removed D1, D2: US1D, Diode_SMD:D_SMA, symbol Diode:US1D
- removed U3: LT3032-12, Package_DFN_QFN:Linear_DE14MA, symbol Regulator_Linear:LT3032-12
- added C23, C24, C25: 10u, Capacitor_SMD:C_0805_2012Metric, symbol Device:C
- added R27: 120k, Resistor_SMD:R_0402_1005Metric, symbol Device:R_US
- added R28: 470k, Resistor_SMD:R_0402_1005Metric, symbol Device:R_US
- added U3: LTC3265xDHC, Package_DFN_QFN:DFN-18-1EP_3x5mm_P0.5mm_EP1.66x4.4mm, symbol OPA_PHONO:LTC3265xDHC
- C14: value 10u -> 1u; footprint Capacitor_SMD:C_0805_2012Metric -> Capacitor_SMD:C_0402_1005Metric
- C15: value 10n -> 10u; footprint Capacitor_SMD:C_0402_1005Metric -> Capacitor_SMD:C_0805_2012Metric
- C16: value 10n -> 1u
- C17, C18: value 10u -> 100n; footprint Capacitor_SMD:C_0805_2012Metric -> Capacitor_SMD:C_0402_1005Metric
- R25: value 4.7R -> 470k; footprint Resistor_SMD:R_2512_6332Metric -> Resistor_SMD:R_0402_1005Metric
- R26: value 4.7R -> ?; footprint Resistor_SMD:R_2512_6332Metric -> Resistor_SMD:R_0402_1005Metric
Connections:
- net REG_P is gone; now on net +12V: R25.1
- net +12V: now also C24.2, U3.17 (LDOP); no longer C15.2, C17.2
- net -12V: now also C25.1, R28.2, U3.7 (LDON); no longer C16.1, C18.1
- net BYPN: now also C18.1, U3.5 (BYPN); no longer C16.2
- net BYPP: now also C17.2, U3.15 (BYPP); no longer C15.1
- net GND: now also C15.1, R26.2, C23.1, C24.1, C25.2, R27.1, U3.12 (RT), U3.14 (MODE), U3.19 (GND); no longer C14.2
- net REG_N renamed ADJP
- net ADJP: now also R25.2, U3.16 (ADJP)
- net REG_P_R renamed VIN
- net VIN: now also U3.13 (ENP), U3.3 (VINP), U3.4 (ENN); no longer R25.2
- net REN_N_R renamed CINVN
- net CINVN: now also U3.9 (CINVN); no longer R26.2
- new net ADJN: R27.2, R28.1, U3.6 (ADJN)
- new net CBSTN: C16.2, U3.1 (CBSTN)
- new net CBSTP: C16.1, U3.2 (CBSTP)
- new net CINVP: C14.2, U3.10 (CINVP)
- new net VOUTN: C15.2, U3.8 (VOUTN)
- new net VOUTP: C23.2, U3.11 (VINN), U3.18 (VOUTP)
Other:
- moved on the sheet: C19, C20, C21, C22, U1E, U2C

Commit message: update layout
Parts:
- added C26, C27, C28, C29, C30: 4.7u, Capacitor_SMD:C_0402_1005Metric, symbol Device:C
- C13, C15, C23, C24, C25: value 10u -> 4.7u; footprint Capacitor_SMD:C_0805_2012Metric -> Capacitor_SMD:C_0402_1005Metric
Connections:
- net +12V: now also C27.2, C29.2; no longer C24.2
- net -12V: now also C28.1, C30.1; no longer C25.1
- net GND: now also C25.1, C26.1, C27.1, C28.2, C29.1, C30.2; no longer C25.2
- net VIN: now also C23.2
- net VOUTN: now also C24.2
- net VOUTP: now also C25.2, C26.2; no longer C23.2

Commit message: add usb c connector
Parts:
- R26: value ? -> 120k
Changed lines of the file:
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@@
       (effects (font (size 1.27 1.27)) (justify left))
     )
-    (property "Value" "?" (id 1) (at 132.08 99.0599 0)
+    (property "Value" "120k" (id 1) (at 132.08 99.0599 0)
       (effects (font (size 1.27 1.27)) (justify left))
     )

Commit message: Update component fields
Parts:
- C19, C20, C21, C22: value 1u -> 4.7u
- R25, R28: MPN (none) -> RC0402FR-07470KL; Manufacturer (none) -> YAGEO
- R26, R27: MPN (none) -> RC0402FR-07120KL; Manufacturer (none) -> YAGEO
- U1: MPN (none) -> OPA1644AID; Manufacturer (none) -> Texas Instruments
- U2: MPN (none) -> OPA1612AID; Manufacturer (none) -> Texas Instruments
- U3: MPN (none) -> LTC3265EDHC#TRPBF; Manufacturer (none) -> Analog Devices Inc.
Changed lines of the file:
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@@
       (effects (font (size 1.27 1.27)) (justify right))
     )
-    (property "Value" "1u" (id 1) (at 184.15 96.5199 0)
+    (property "Value" "4.7u" (id 1) (at 184.15 96.5199 0)
       (effects (font (size 1.27 1.27)) (justify right))
     )
@@
     )
     (property "Datasheet" "~" (id 3) (at 129.54 97.79 0)
+      (effects (font (size 1.27 1.27)) hide)
+    )
+    (property "Description" "RES SMD 120K OHM 1% 1/16W 0402" (id 4) (at 129.54 97.79 0)
+      (effects (font (size 1.27 1.27)) hide)
+    )
+    (property "MPN" "RC0402FR-07120KL" (id 5) (at 129.54 97.79 0)
+      (effects (font (size 1.27 1.27)) hide)
+    )
+    (property "Manufacturer" "YAGEO" (id 6) (at 129.54 97.79 0)
       (effects (font (size 1.27 1.27)) hide)
     )
@@
       (effects (font (size 1.27 1.27)) hide)
     )
+    (property "Description" "RES SMD 120K OHM 1% 1/16W 0402" (id 4) (at 129.54 105.41 0)
+      (effects (font (size 1.27 1.27)) hide)
+    )
+    (property "MPN" "RC0402FR-07120KL" (id 5) (at 129.54 105.41 0)
+      (effects (font (size 1.27 1.27)) hide)
+    )
+    (property "Manufacturer" "YAGEO" (id 6) (at 129.54 105.41 0)
+      (effects (font (size 1.27 1.27)) hide)
+    )
     (pin "1")
     (pin "2")
@@
       (effects (font (size 1.27 1.27)) hide)
     )
+    (property "Description" "IC AUDIO 4 CIRCUIT 14SOIC" (id 4) (at 193.04 100.33 0)
+      (effects (font (size 1.27 1.27)) hide)
+    )
+    (property "MPN" "OPA1644AID" (id 5) (at 193.04 100.33 0)
+      (effects (font (size 1.27 1.27)) hide)
+    )
+    (property "Manufacturer" "Texas Instruments" (id 6) (at 193.04 100.33 0)
+      (effects (font (size 1.27 1.27)) hide)
+    )
     (pin "11")
     (pin "4")
@@
       (effects (font (size 1.27 1.27)) (justify right))
     )
-    (property "Value" "1u" (id 1) (at 208.28 107.9499 0)
+    (property "Value" "4.7u" (id 1) (at 208.28 107.9499 0)
       (effects (font (size 1.27 1.27)) (justify right))
     )
@@
       (effects (font (size 1.27 1.27)) (justify right))
     )
-    (property "Value" "1u" (id 1) (at 184.15 109.2199 0)
+    (property "Value" "4.7u" (id 1) (at 184.15 109.2199 0)
       (effects (font (size 1.27 1.27)) (justify right))
     )
@@
     )
     (property "Datasheet" "https://www.analog.com/media/en/technical-documentation/data-sheets/3265fa.pdf" (id 3) (at 83.82 68.58 0)
+      (effects (font (size 1.27 1.27)) hide)
+    )
+    (property "Description" "IC REG CHARGE PUMP INV 18DFN" (id 4) (at 83.82 68.58 0)
+      (effects (font (size 1.27 1.27)) hide)
+    )
+    (property "MPN" "LTC3265EDHC#TRPBF" (id 5) (at 83.82 68.58 0)
+      (effects (font (size 1.27 1.27)) hide)
+    )
+    (property "Manufacturer" "Analog Devices Inc." (id 6) (at 83.82 68.58 0)
       (effects (font (size 1.27 1.27)) hide)
     )
@@
       (effects (font (size 1.27 1.27)) hide)
     )
+    (property "Description" "RES 470K OHM 1% 1/16W 0402" (id 4) (at 129.54 115.57 0)
+      (effects (font (size 1.27 1.27)) hide)
+    )
+    (property "MPN" "RC0402FR-07470KL" (id 5) (at 129.54 115.57 0)
+      (effects (font (size 1.27 1.27)) hide)
+    )
+    (property "Manufacturer" "YAGEO" (id 6) (at 129.54 115.57 0)
+      (effects (font (size 1.27 1.27)) hide)
+    )
     (pin "1")
     (pin "2")
@@
       (effects (font (size 1.27 1.27)) hide)
     )
+    (property "Description" "RES 470K OHM 1% 1/16W 0402" (id 4) (at 129.54 87.63 0)
+      (effects (font (size 1.27 1.27)) hide)
+    )
+    (property "MPN" "RC0402FR-07470KL" (id 5) (at 129.54 87.63 0)
+      (effects (font (size 1.27 1.27)) hide)
+    )
+    (property "Manufacturer" "YAGEO" (id 6) (at 129.54 87.63 0)
+      (effects (font (size 1.27 1.27)) hide)
+    )
     (pin "1")
     (pin "2")
@@
       (effects (font (size 1.27 1.27)) (justify right))
     )
-    (property "Value" "1u" (id 1) (at 208.28 96.5199 0)
+    (property "Value" "4.7u" (id 1) (at 208.28 96.5199 0)
       (effects (font (size 1.27 1.27)) (justify right))
     )
@@
       (effects (font (size 1.27 1.27)) hide)
     )
+    (property "Description" "IC AUDIO 2 CIRCUIT 8SOIC" (id 4) (at 217.17 100.33 0)
+      (effects (font (size 1.27 1.27)) hide)
+    )
+    (property "MPN" "OPA1612AID" (id 5) (at 217.17 100.33 0)
+      (effects (font (size 1.27 1.27)) hide)
+    )
+    (property "Manufacturer" "Texas Instruments" (id 6) (at 217.17 100.33 0)
+      (effects (font (size 1.27 1.27)) hide)
+    )

Commit message: routed all nets
Parts:
- removed C15, C25, C29, C30: 4.7u, Capacitor_SMD:C_0402_1005Metric, symbol Device:C
- C13, C19, C20, C21, C22: value 4.7u -> 1u; MPN (none) -> GRM155R61E105KA12D; Manufacturer (none) -> Murata Electronics
- C14, C16: MPN (none) -> GRM155R61E105KA12D; Manufacturer (none) -> Murata Electronics
- C17, C18: value 100n -> 1u; MPN (none) -> GRM155R61E105KA12D; Manufacturer (none) -> Murata Electronics
- C23, C24, C26, C27, C28: value 4.7u -> 10u; footprint Capacitor_SMD:C_0402_1005Metric -> Capacitor_SMD:C_0805_2012Metric; MPN (none) -> GRM21BR61C106KE15L; Manufacturer (none) -> Murata Electronics
Connections:
- net VIN: no longer C13.2
- net VOUTP: now also C13.2

Commit message: simplify BOM
Parts:
- C13, C14, C16, C17, C18, C19, C20, C21, C22: Rating (none) -> 25V; Size (none) -> 0402; Tolerance (none) -> X5R
- C23, C24, C26, C27, C28: Rating (none) -> 16V; Size (none) -> 0805; Tolerance (none) -> X5R
- R25, R28: value 470k -> 20.5k; MPN RC0402FR-07470KL -> RC0402FR-0720K5L; Size (none) -> 0402; Tolerance (none) -> 1%
- R26, R27: value 120k -> 5.1k; MPN RC0402FR-07120KL -> RC0402FR-075K1L; Size (none) -> 0402; Tolerance (none) -> 1%
Connections:
- net +12V renamed +6V
- net -12V renamed -6V
Other:
- note added: "LDO 50mA"
- moved on the sheet: C19, C20, C21, C22, C27, C28, U1E, U2C

Commit message: Generate Gerbers
Parts:
- added C15, C25: 10u, Capacitor_SMD:C_0805_2012Metric, symbol Device:C
Connections:
- net +6V: now also C15.2
- net -6V: now also C25.1
- net GND: now also C15.1, C25.2
Other:
- moved on the sheet: C19, C20, C21, C22, U1E, U2C
