File: PCB/RIAA_PHONO.kicad_sch (KiCad schematic)
At the start: 20 parts, among them U1 OPA1644AxD, U2 OPA1612AxD

Commit message: differential amp initial changes
Parts:
- removed R3: 499R, Resistor_SMD:R_0402_1005Metric, symbol Device:R_US
- added R31, R32, R33: 16k, Resistor_SMD:R_0402_1005Metric, symbol Device:R_US
- added R34: 499R, Resistor_SMD:R_0402_1005Metric, symbol Device:R_US
- added U4: OPA1612AxD, Package_SO:SOIC-8_3.9x4.9mm_P1.27mm, symbol Amplifier_Operational:OPA1612AxD
- renumbered C4 to C10, C5 to C11, C6 to C12, C1 to C7, C2 to C8, C3 to C9, R1 to R13, R2 to R14, R4 to R16, R5 to R17, R7 to R19, R9 to R21, R10 to R22, R11 to R23, R12 to R24, R8 to R6
Connections:
- net FBTRIM: now also U4.2 (-); no longer U1.2 (-)
- net GND: now also R33.2; no longer C7.2, R13.1
- net OUT_RC: now also U4.3 (+); no longer U1.3 (+)
- net TRIM: now also U4.1; no longer U1.1
- net FB1 renamed FB1P
- net FB1P: now also R31.1, R34.2
- net IN renamed INP
- new net FB1N: R32.2, R33.1, R34.1, U1.2 (-)
- new net INN: C7.2, R13.1, U1.3 (+)
- new net OUT1B: R31.2, R32.1, U1.1
